File: Kicad/BatteryCharger.kicad_sch (KiCad schematic)
At the start: 28 parts, among them IC1 AP9214L-AN-HSBR-7, IC2 TPS61085TDGKR

Commit message: New HW v1.25 release
Parts:
- IC1: value AP9214L-AN-HSBR-7 -> AP9214L-AD-HSBR-7
Other:
- note added: "BMS CIRCUIT: Charging: -TP4056 as a well-known charging IC, up to 500mA with a 2.1K PROG resistor. -We do not use NTC for the battery in order to save costs. Protection IC: -AP9214L-AD-HSBR-7 as main chip. It disconnects the ground of the battery from the rest of the circuit. -4.325V max voltage to 2.9V min voltage (protections). -Auto-release. Boost Converter: -TPS61085TDGKR as main chip. -Toggl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"
- note removed: "BMS CIRCUIT: Charging: -TP4056 as a well-known charging IC, up to 500mA with a 2.1K PROG resistor. -We do not use NTC for the battery in order to save costs. Protection IC: -AP9214L-AN-HSBR-7 as main chip. It disconnects the ground of the battery from the rest of the circuit. -4.225V max voltage to 3.2V min voltage (protections). -Auto-release. Boost Converter: -TPS61085TDGKR as main chip. -Toggl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"
Changed lines of the file:
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@@
     (effects (font (size 1.27 1.27)) (justify left bottom))
   )
-  (text "BMS CIRCUIT:\nCharging:\n-TP4056 as a well-known charging IC, up to 500mA with a 2.1K PROG resistor.\n-We do not use NTC for the battery in order to save costs.\n\nProtection IC:\n-AP9214L-AN-HSBR-7 as main chip. It disconnects the ground of the battery from the rest of the circuit.\n-4.225V max voltage to 3.2V min voltage (protections).\n-Auto-release. \n\nBoost Converter:\n-TPS61085TDGKR as main chip. \n-Toggle Switch.\n-5V fix output voltage. 0.6A maximum output current \n\nUSB type C \n-Type C connector.\n-Only for charging"
+  (text "BMS CIRCUIT:\nCharging:\n-TP4056 as a well-known charging IC, up to 500mA with a 2.1K PROG resistor.\n-We do not use NTC for the battery in order to save costs.\n\nProtection IC:\n-AP9214L-AD-HSBR-7 as main chip. It disconnects the ground of the battery from the rest of the circuit.\n-4.325V max voltage to 2.9V min voltage (protections).\n-Auto-release. \n\nBoost Converter:\n-TPS61085TDGKR as main chip. \n-Toggle Switch.\n-5V fix output voltage. 0.6A maximum output current \n\nUSB type C \n-Type C connector.\n-Only for charging"
     (at 21.59 182.88 0)
     (effects (font (size 1.27 1.27)) (justify left bottom))
@@
       (effects (font (size 1.27 1.27)))
     )
-    (property "Value" "AP9214L-AN-HSBR-7" (at 90.17 107.3404 0)
-      (effects (font (size 1.27 1.27)))
-    )
+    (property "Value" "AP9214L-AD-HSBR-7" (at 90.17 107.3404 0)
+      (effects (font (size 1.27 1.27)))
+    )

Commit message: Bill Of Materials
Parts:
- C14: renamed from C_10u_1; value GCG21BR71H154KA01K -> 10uF
- R58: renamed from R_2k_1; value KTR10EZPF4220 -> 2k
- R59: renamed from R_1k_1; value KTR10EZPF4220 -> 1k
- R60: renamed from R_1k_2; value KTR10EZPF4220 -> 1k
- R61: renamed from R_5.1k_1; value KTR10EZPF4220 -> 5.1k
- R62: renamed from R_5.1_1; value KTR10EZPF4220 -> 5.1k
Changed lines of the file:
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@@
 		(on_board yes)
 		(dnp no)
-		(property "Reference" "R_2k_1"
-			(at 58.42 42.3418 0)
-			(effects
-				(font
-					(size 1.27 1.27)
-				)
-			)
-		)
-		(property "Value" "KTR10EZPF4220"
-			(at 58.42 42.3164 0)
-			(effects
-				(font
-					(size 1.27 1.27)
-				)
-				(hide yes)
+		(property "Reference" "R58"
+			(at 56.134 42.418 0)
+			(effects
+				(font
+					(size 1.27 1.27)
+				)
+			)
+		)
+		(property "Value" "2k"
+			(at 60.96 42.418 0)
+			(effects
+				(font
+					(size 1.27 1.27)
+				)
 			)
 		)
@@
 			(project "PicBytesMicro"
 				(path "/36e2b0cc-9d11-4a29-a898-cd33b5ef9720/00000000-0000-0000-0000-00006009e6f5"
-					(reference "R_2k_1")
+					(reference "R58")
 					(unit 1)
 				)
@@
 		(on_board yes)
 		(dnp no)
-		(property "Reference" "C_10u_1"
+		(property "Reference" "C14"
 			(at 66.7512 57.15 0)
 			(effects
@@
 			)
 		)
-		(property "Value" "GCG21BR71H154KA01K"
+		(property "Value" "10uF"
 			(at 66.7512 58.293 90)
 			(effects
@@
 			(project "PicBytesMicro"
 				(path "/36e2b0cc-9d11-4a29-a898-cd33b5ef9720/00000000-0000-0000-0000-00006009e6f5"
-					(reference "C_10u_1")
+					(reference "C14")
 					(unit 1)
 				)
@@
 		(on_board yes)
 		(dnp no)
-		(property "Reference" "R_5.1k_1"
-			(at 186.69 34.7218 0)
-			(effects
-				(font
-					(size 1.27 1.27)
-				)
-			)
-		)
-		(property "Value" "KTR10EZPF4220"
-			(at 186.69 34.6964 0)
-			(effects
-				(font
-					(size 1.27 1.27)
-				)
-				(hide yes)
+		(property "Reference" "R61"
+			(at 182.372 34.544 0)
+			(effects
+				(font
+					(size 1.27 1.27)
+				)
+			)
+		)
+		(property "Value" "5.1k"
+			(at 188.722 35.306 0)
+			(effects
+				(font
+					(size 1.27 1.27)
+				)
 			)
 		)
@@
 			(project "PicBytesMicro"
 				(path "/36e2b0cc-9d11-4a29-a898-cd33b5ef9720/00000000-0000-0000-0000-00006009e6f5"
-					(reference "R_5.1k_1")
+					(reference "R61")
 					(unit 1)
 				)
@@
 		(on_board yes)
 		(dnp no)
-		(property "Reference" "R_5.1_1"
-			(at 186.69 42.3418 0)
-			(effects
-				(font
-					(size 1.27 1.27)
-				)
-			)
-		)
-		(property "Value" "KTR10EZPF4220"
-			(at 186.69 42.3164 0)
-			(effects
-				(font
-					(size 1.27 1.27)
-				)
-				(hide yes)
+		(property "Reference" "R62"
+			(at 186.182 42.418 0)
+			(effects
+				(font
+					(size 1.27 1.27)
+				)
+			)
+		)
+		(property "Value" "5.1k"
+			(at 186.69 48.006 0)
+			(effects
+				(font
+					(size 1.27 1.27)
+				)
 			)
 		)
@@
 			(project "PicBytesMicro"
 				(path "/36e2b0cc-9d11-4a29-a898-cd33b5ef9720/00000000-0000-0000-0000-00006009e6f5"
-					(reference "R_5.1_1")
+					(reference "R62")
 					(unit 1)
 				)
@@
 		(on_board yes)
 		(dnp no)
-		(property "Reference" "R_1k_1"
+		(property "Reference" "R59"
 			(at 108.9152 58.42 0)
 			(effects
@@
 			)
 		)
-		(property "Value" "KTR10EZPF4220"
-			(at 108.9152 59.563 90)
-			(effects
-				(font
-					(size 1.27 1.27)
-				)
-				(justify left)
-				(hide yes)
+		(property "Value" "1k"
+			(at 107.95 55.88 90)
+			(effects
+				(font
+					(size 1.27 1.27)
+				)
+				(justify left)
 			)
 		)
@@
 			(project "PicBytesMicro"
 				(path "/36e2b0cc-9d11-4a29-a898-cd33b5ef9720/00000000-0000-0000-0000-00006009e6f5"
-					(reference "R_1k_1")
+					(reference "R59")
 					(unit 1)
 				)
@@
 		(on_board yes)
 		(dnp no)
-		(property "Reference" "R_1k_2"
+		(property "Reference" "R60"
 			(at 117.8052 58.42 0)
 			(effects
@@
 			)
 		)
-		(property "Value" "KTR10EZPF4220"
-			(at 117.8052 59.563 90)
-			(effects
-				(font
-					(size 1.27 1.27)
-				)
-				(justify left)
-				(hide yes)
+		(property "Value" "1k"
+			(at 117.094 55.88 90)
+			(effects
+				(font
+					(size 1.27 1.27)
+				)
+				(justify left)
 			)
 		)
@@
 			(project "PicBytesMicro"
 				(path "/36e2b0cc-9d11-4a29-a898-cd33b5ef9720/00000000-0000-0000-0000-00006009e6f5"
-					(reference "R_1k_2")
+					(reference "R60")
 					(unit 1)
 				)
