File: Kicad/PicBytesMicro.kicad_sch (KiCad schematic)
At the start: 9 parts, among them J1 TC2030-MCP-NL, Y1 CX2520DB12000D0GPSC1

Commit message: no message
Parts:
- gave numbers to parts that had none: 2

Commit message: Bill Of Materials
Parts:
- C12: renamed from C_22p_1; value GCG21BR71H154KA01K -> 22pF
- C13: renamed from C_22p_2; value GCG21BR71H154KA01K -> 22pF
- PIC18F4550: renamed from PIC18F45K1; value PIC18F45K50-I_PT -> PIC18F4550-I_PT
- R45: renamed from R_10k_1; value KTR10EZPF4220 -> 10k
- R7: renamed from R4K7_1; value KTR10EZPF4220 -> 4k7
Changed lines of the file:
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@@
 		(on_board yes)
 		(dnp no)
-		(property "Reference" "C_22p_1"
+		(property "Reference" "C12"
 			(at 239.4712 57.15 0)
 			(effects
@@
 			)
 		)
-		(property "Value" "GCG21BR71H154KA01K"
-			(at 239.4712 58.293 90)
-			(effects
-				(font
-					(size 1.27 1.27)
-				)
-				(justify left)
-				(hide yes)
+		(property "Value" "22pF"
+			(at 231.648 55.372 90)
+			(effects
+				(font
+					(size 1.27 1.27)
+				)
+				(justify left)
 			)
 		)
@@
 			(project "PicBytesMicro"
 				(path "/36e2b0cc-9d11-4a29-a898-cd33b5ef9720"
-					(reference "C_22p_1")
+					(reference "C12")
 					(unit 1)
 				)
@@
 		(on_board yes)
 		(dnp no)
-		(property "Reference" "C_22p_2"
+		(property "Reference" "C13"
 			(at 245.8212 57.15 0)
 			(effects
@@
 			)
 		)
-		(property "Value" "GCG21BR71H154KA01K"
-			(at 245.8212 58.293 90)
-			(effects
-				(font
-					(size 1.27 1.27)
-				)
-				(justify left)
-				(hide yes)
+		(property "Value" "22pF"
+			(at 245.364 62.23 90)
+			(effects
+				(font
+					(size 1.27 1.27)
+				)
+				(justify left)
 			)
 		)
@@
 			(project "PicBytesMicro"
 				(path "/36e2b0cc-9d11-4a29-a898-cd33b5ef9720"
-					(reference "C_22p_2")
+					(reference "C13")
 					(unit 1)
 				)
@@
 		(on_board yes)
 		(dnp no)
-		(property "Reference" "R_10k_1"
+		(property "Reference" "R45"
 			(at 204.47 135.89 0)
 			(effects
@@
 			)
 		)
-		(property "Value" "KTR10EZPF4220"
-			(at 204.47 135.0264 0)
-			(effects
-				(font
-					(size 1.27 1.27)
-				)
-				(hide yes)
+		(property "Value" "10k"
+			(at 204.724 141.224 0)
+			(effects
+				(font
+					(size 1.27 1.27)
+				)
 			)
 		)
@@
 			(project "PicBytesMicro"
 				(path "/36e2b0cc-9d11-4a29-a898-cd33b5ef9720"
-					(reference "R_10k_1")
+					(reference "R45")
 					(unit 1)
 				)
@@
 		(on_board yes)
 		(dnp no)
-		(property "Reference" "R4K7_1"
+		(property "Reference" "R7"
 			(at 120.65 55.245 0)
 			(effects
@@
 			)
 		)
-		(property "Value" "KTR10EZPF4220"
+		(property "Value" "4k7"
 			(at 120.65 57.5564 0)
 			(effects
@@
 			(project "PicBytesMicro"
 				(path "/36e2b0cc-9d11-4a29-a898-cd33b5ef9720"
-					(reference "R4K7_1")
+					(reference "R7")
 					(unit 1)
 				)
@@
 		(on_board yes)
 		(dnp no)
-		(property "Reference" "PIC18F45K1"
+		(property "Reference" "PIC18F4550"
 			(at 180.34 55.88 0)
 			(effects
@@
 			)
 		)
-		(property "Value" "PIC18F45K50-I_PT"
+		(property "Value" "PIC18F4550-I_PT"
 			(at 234.7976 82.423 0)
 			(effects
@@
 			(project "PicBytesMicro"
 				(path "/36e2b0cc-9d11-4a29-a898-cd33b5ef9720"
-					(reference "PIC18F45K1")
+					(reference "PIC18F4550")
 					(unit 1)
 				)
