File: Kicad/Screen.kicad_sch (KiCad schematic)
At the start: 226 parts, among them Q1 SMMBT5551LT1G, Q10 SMMBT5551LT1G, Q11 SMMBT5551LT1G, Q12 SMMBT5551LT1G, Q13 SMMBT5551LT1G, Q14 SMMBT5551LT1G, Q15 SMMBT5551LT1G, Q16 SMMBT5551LT1G, Q17 SMMBT5551LT1G, Q18 SMMBT5551LT1G, Q19 SMMBT5551LT1G, Q2 SMMBT5551LT1G, Q20 SMMBT5551LT1G, Q21 SMMBT5551LT1G, Q22 SMMBT5551LT1G, Q23 SMMBT5551LT1G, Q24 SMMBT5551LT1G, Q25 SMMBT5551LT1G, Q26 SMMBT5551LT1G, Q27 SMMBT5551LT1G, Q28 SMMBT5551LT1G, Q3 SMMBT5551LT1G, Q4 SMMBT5551LT1G, Q5 SMMBT5551LT1G, Q6 SMMBT5551LT1G, Q7 SMMBT5551LT1G, Q8 SMMBT5551LT1G, Q9 SMMBT5551LT1G

Commit message: New V1.2 Hardware Release
Parts:
- renumbered Q9 to Q10, Q10 to Q11, Q11 to Q12, Q12 to Q13, Q13 to Q14, Q14 to Q15, Q15 to Q16, Q16 to Q17, Q17 to Q18, Q18 to Q19, Q1 to Q2, Q19 to Q20, Q20 to Q21, Q21 to Q22, Q22 to Q23, Q23 to Q24, Q24 to Q25, Q25 to Q26, Q26 to Q27, Q27 to Q28, Q28 to Q29, Q2 to Q3, Q3 to Q4, Q4 to Q5, Q5 to Q6, Q6 to Q7, Q7 to Q8, Q8 to Q9, R4K7_9 to R4K7_10, R4K7_10 to R4K7_11, R4K7_11 to R4K7_12, R4K7_12 to R4K7_13, R4K7_13 to R4K7_14, R4K7_14 to R4K7_15, R4K7_15 to R4K7_16, R4K7_16 to R4K7_17, R4K7_17 to R4K7_18, R4K7_18 to R4K7_19, R4K7_1 to R4K7_2, R4K7_19 to R4K7_20, R4K7_20 to R4K7_21, R4K7_21 to R4K7_22, R4K7_22 to R4K7_23, R4K7_23 to R4K7_24, R4K7_24 to R4K7_25, R4K7_25 to R4K7_26, R4K7_26 to R4K7_27, R4K7_27 to R4K7_28, R4K7_28 to R4K7_29, R4K7_2 to R4K7_3, R4K7_3 to R4K7_4, R4K7_4 to R4K7_5, R4K7_5 to R4K7_6, R4K7_6 to R4K7_7, R4K7_7 to R4K7_8, R4K7_8 to R4K7_9

Commit message: Bill Of Materials
Parts:
- R10: renamed from R4K7_4; value KTR10EZPF4220 -> 4k7
- R11: renamed from R4K7_5; value KTR10EZPF4220 -> 4k7
- R12: renamed from R4K7_6; value KTR10EZPF4220 -> 4k7
- R13: renamed from R4K7_7; value KTR10EZPF4220 -> 4k7
- R14: renamed from R220_1; value KTR10EZPF4220 -> 220
- R15: renamed from R220_2; value KTR10EZPF4220 -> 220
- R16: renamed from R4K7_8; value KTR10EZPF4220 -> 4k7
- R17: renamed from R4K7_9; value KTR10EZPF4220 -> 4k7
- R18: renamed from R4K7_10; value KTR10EZPF4220 -> 4k7
- R19: renamed from R4K7_11; value KTR10EZPF4220 -> 4k7
- R20: renamed from R220_3; value KTR10EZPF4220 -> 220
- R21: renamed from R220_4; value KTR10EZPF4220 -> 220
- R22: renamed from R4K7_12; value KTR10EZPF4220 -> 4k7
- R220: renamed from R220_8; value KTR10EZPF4220 -> 220
- R23: renamed from R4K7_13; value KTR10EZPF4220 -> 4k7
- R24: renamed from R4K7_14; value KTR10EZPF4220 -> 4k7
- R25: renamed from R4K7_15; value KTR10EZPF4220 -> 4k7
- R26: renamed from R4K7_16; value KTR10EZPF4220 -> 4k7
- R27: renamed from R4K7_17; value KTR10EZPF4220 -> 4k7
- R28: renamed from R4K7_18; value KTR10EZPF4220 -> 4k7
- R29: renamed from R4K7_19; value KTR10EZPF4220 -> 4k7
- R30: renamed from R220_5; value KTR10EZPF4220 -> 220
- R31: renamed from R220_6; value KTR10EZPF4220 -> 220
- R32: renamed from R4K7_20; value KTR10EZPF4220 -> 4k7
- R33: renamed from R4K7_21; value KTR10EZPF4220 -> 4k7
- R34: renamed from R4K7_22; value KTR10EZPF4220 -> 4k7
- R35: renamed from R4K7_23; value KTR10EZPF4220 -> 4k7
- R36: renamed from R220_7; value KTR10EZPF4220 -> 220
- R37: renamed from R4K7_24; value KTR10EZPF4220 -> 4k7
- R38: renamed from R4K7_25; value KTR10EZPF4220 -> 4k7
- R39: renamed from R4K7_26; value KTR10EZPF4220 -> 4k7
- R40: renamed from R4K7_27; value KTR10EZPF4220 -> 4k7
- R41: renamed from R220_9; value KTR10EZPF4220 -> 220
- R42: renamed from R220_10; value KTR10EZPF4220 -> 220
- R43: renamed from R4K7_28; value KTR10EZPF4220 -> 4k7
- R44: renamed from R4K7_29; value KTR10EZPF4220 -> 4k7
- R8: renamed from R4K7_2; value KTR10EZPF4220 -> 4k7
- R9: renamed from R4K7_3; value KTR10EZPF4220 -> 4k7
